File: Hardware/Power.kicad_sch (KiCad schematic)
At the start: 16 parts, among them U1 LV2862YDDCR, U2 AMS1117-3.3

Commit message: Re-layout
Parts:
- added D6, D7: BAT54WS, Diode_SMD:D_SOD-323_HandSoldering, symbol Device:D_Schottky_Small
Connections:
- net +12VA: now also D6.2 (A); no longer C5.2, U2.3 (VI)
- new net: C5.2, D6.1 (K), D7.1 (K), U2.3 (VI)
- new net 3V3regIn: D7.2 (A)
Changed lines of the file:
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@@
+    (stroke (width 0) (type default))
+  )
+  (wire (pts (xy 205.74 96.52) (xy 205.74 101.6))
     (stroke (width 0) (type default))
   )
@@
     (stroke (width 0) (type default))
   )
-  (wire (pts (xy 171.45 101.6) (xy 205.74 101.6))
+  (wire (pts (xy 171.45 101.6) (xy 185.42 101.6))
     (stroke (width 0) (type default))
   )
@@
     (stroke (width 0) (type default))
   )
+  (wire (pts (xy 205.74 88.9) (xy 205.74 91.44))
+    (stroke (width 0) (type default))
+  )
   (wire (pts (xy 166.37 77.47) (xy 171.45 77.47))
     (stroke (width 0) (type default))
@@
   )
   (wire (pts (xy 156.21 91.44) (xy 156.21 85.09))
+    (stroke (width 0) (type default))
+  )
+  (wire (pts (xy 190.5 101.6) (xy 205.74 101.6))
     (stroke (width 0) (type default))
   )
@@
     (effects (font (size 1.27 1.27)) (justify left bottom))
   )
+  (hierarchical_label "3V3regIn" (shape input) (at 205.74 88.9 90) (fields_autoplaced)
+    (effects (font (size 1.27 1.27)) (justify left))
+  )
   (hierarchical_label "GND" (shape passive) (at 175.26 127 0) (fields_autoplaced)
     (effects (font (size 1.27 1.27)) (justify left))
@@
         (path "/201932c1-739b-4a93-a19c-4122cdfb0c30/06542b34-8b5c-4664-a2e3-49fb4aa24614"
           (reference "D2") (unit 1)
+        )
+      )
+    )
+  )
+  (symbol (lib_id "Device:D_Schottky_Small") (at 205.74 93.98 90) (unit 1)
+    (in_bom yes) (on_board yes) (dnp no)
+    (property "Reference" "D7" (at 203.2 93.599 90)
+      (effects (font (size 1.27 1.27)) (justify left))
+    )
+    (property "Value" "BAT54WS" (at 203.2 95.25 90)
+      (effects (font (size 1.27 1.27)) (justify left))
+    )
+    (property "Footprint" "Diode_SMD:D_SOD-323_HandSoldering" (at 205.74 93.98 90)
+      (effects (font (size 1.27 1.27)) hide)
+    )
+    (property "Datasheet" "~" (at 205.74 93.98 90)
+      (effects (font (size 1.27 1.27)) hide)
+    )
+    (pin "1")
+    (pin "2")
+    (instances
+      (project "Morten-sol-vindue"
+        (path "/201932c1-739b-4a93-a19c-4122cdfb0c30/06542b34-8b5c-4664-a2e3-49fb4aa24614"
+          (reference "D7") (unit 1)
         )
       )
@@
         )
       )
+    )
+  )
+  (symbol (lib_id "Device:D_Schottky_Small") (at 187.96 101.6 0) (mirror y) (unit 1)
+    (in_bom yes) (on_board yes) (dnp no) (fields_autoplaced)
+    (property "Reference" "D6" (at 188.214 96.52 0)
+      (effects (font (size 1.27 1.27)))
+    )
+    (property "Value" "BAT54WS" (at 188.214 99.06 0)
+      (effects (font (size 1.27 1.27)))
+    )
+    (property "Footprint" "Diode_SMD:D_SOD-323_HandSoldering" (at 187.96 101.6 90)
+      (effects (font (size 1.27 1.27)) hide)
+    )
+    (property "Datasheet" "~" (at 187.96 101.6 90)
+      (effects (font (size 1.27 1.27)) hide)
+    )
+    (pin "1")
+    (pin "2")
+    (instances
+      (project "Morten-sol-vindue"
+        (path "/201932c1-739b-4a93-a19c-4122cdfb0c30/06542b34-8b5c-4664-a2e3-49fb4aa24614"
+          (reference "D6") (unit 1)
+        )
+      )
