File: Hardware/Power.kicad_sch (KiCad schematic)
At the start: 18 parts, among them U1 LV2862YDDCR, U2 AMS1117-3.3

Commit message: Full functionality
Parts:
- C2: value 1uF 25V -> 10nF 25v
- R3: value 100R -> 120R
Changed lines of the file:
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@@
       (effects (font (size 1.27 1.27)) (justify right))
     )
-    (property "Value" "100R" (at 168.91 89.535 0)
+    (property "Value" "120R" (at 168.91 89.535 0)
       (effects (font (size 1.27 1.27)) (justify right))
     )
@@
   (symbol (lib_id "Device:C_Small") (at 149.86 77.47 90) (mirror x) (unit 1)
     (in_bom yes) (on_board yes) (dnp no) (fields_autoplaced)
-    (property "Reference" "C2" (at 149.8663 82.55 90)
+    (property "Reference" "C2" (at 149.8663 71.12 90)
       (effects (font (size 1.27 1.27)))
     )
-    (property "Value" "1uF 25V" (at 149.8663 80.01 90)
+    (property "Value" "10nF 25v" (at 149.8663 73.66 90)
       (effects (font (size 1.27 1.27)))
     )
